File: pi-hat/kicad/PiHat.kicad_pcb (KiCad board)
At the start: 2 copper layers, 49.8 x 63 mm, 15 parts, among them J1 Raspberry_Pi_2_3, J2 Power, J3 HDMI board, J4 Fan, J5 CNC, J6 IDC16, J7 UVPanel, J8 Pro Power, J9 Buzzer, Q1 BD139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

Commit message: Updated PiHat schematic to reflect proper values to read z-probe
Parts:
- R1: value 2K2 -> 1K8
- R2: value 3K3 -> 20K
Changed lines of the file:
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@@
       (effects (font (size 1 1) (thickness 0.15)))
     )
-    (fp_text value 3K3 (at 5 0 90) (layer F.SilkS)
+    (fp_text value 20K (at 5 0 90) (layer F.SilkS)
       (effects (font (size 1 1) (thickness 0.15)))
     )
@@
       (effects (font (size 1 1) (thickness 0.15)))
     )
-    (fp_text value 2K2 (at 5.25 0 90) (layer F.SilkS)
+    (fp_text value 1K8 (at 5.25 0 90) (layer F.SilkS)
       (effects (font (size 1 1) (thickness 0.15)))
     )
