File: test/Test.sch (KiCad schematic (older format))
At the start: 15 parts, among them J1 Raspberry_Pi_2_3, J2 Power, J3 HDMI board, J4 Fan, J5 CNC, J6 IDC16, J7 UVPanel, J8 Pro Power, J9 Buzzer, Q1 BD139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

Commit message: Do not use pcb2gcode tool change gcode
pcb2gcode generates tool change code. Remove that at runtime, as the mill is already prepped.
Parts:
- removed D1: 1N4001, Diode_THT:D_DO-41_SOD81_P10.16mm_Horizontal, symbol Diode:1N4001
- removed J1: Raspberry_Pi_2_3, pcb_etcher:PinSocket_2x20_P2.54mm_BacksideMount, symbol Connector:Raspberry_Pi_2_3
- removed J2: Power, Connector_JST:JST_XH_B2B-XH-A_1x02_P2.50mm_Vertical, symbol Connector_Generic:Conn_01x02
- removed J3: HDMI board, Connector_JST:JST_XH_B2B-XH-A_1x02_P2.50mm_Vertical, symbol Connector_Generic:Conn_01x02
- removed J4: Fan, Connector_JST:JST_XH_B2B-XH-A_1x02_P2.50mm_Vertical, symbol Connector_Generic:Conn_01x02
- removed J6: IDC16, Connector_IDC:IDC-Header_2x08_P2.54mm_Vertical, symbol Connector_Generic:Conn_02x08_Odd_Even
- removed J7: UVPanel, Connector_JST:JST_XH_B5B-XH-A_1x05_P2.50mm_Vertical, symbol Connector_Generic:Conn_01x05
- removed J8: Pro Power, Connector_JST:JST_XH_B2B-XH-A_1x02_P2.50mm_Vertical, symbol Connector_Generic:Conn_01x02
- removed J9: Buzzer, Connector_PinHeader_2.54mm:PinHeader_2x01_P2.54mm_Vertical, symbol Connector_Generic:Conn_01x02
- removed R1: 1K8, Resistor_THT:R_Axial_DIN0207_L6.3mm_D2.5mm_P10.16mm_Horizontal, symbol Device:R
- removed R2: 20K, Resistor_THT:R_Axial_DIN0207_L6.3mm_D2.5mm_P10.16mm_Horizontal, symbol Device:R
- removed R3: 1k, Resistor_THT:R_Axial_DIN0207_L6.3mm_D2.5mm_P10.16mm_Horizontal, symbol Device:R_Small_US
- removed U1: AMZ_3A_MOD, jkoz_custom:Amazon_3A_Power_Module, symbol jkoz_custom:AMZ_3A_MOD
Connections:
- net labels removed: +24V, +3.3V, Buzzer, CS, DC, GND, MISO, MOSI, RESET, SCL, SDA, SLCK, T_CS, T_IRQ, UVControl, ZProbe3V3, ZProbeIn
- wire segments 16 -> 0
- no-connect marks 26 -> 3
Other:
- note removed: "12v_-_24v_Regulated_Power"
