File: hardware/pro-controller/pi-hat/kicad/PiHatPro.kicad_pcb (KiCad board)
At the start: 4 copper layers, 49.8 x 63 mm, 11 parts, among them J1 Raspberry_Pi_2_3, J2 Power, J3 UVPanel, J4 Joystick, J5 CNC, J9 Buzzer, U1 AMZ_3A_MOD, U2 ADS1115

Commit message: Pi Hat is now single sided
Pi Hat Rev 3.1 is now completely single sided for easier DIY fabrication
Routing:
- net +3V3: track 64.1 -> 44.7 mm
- net GND: track 257.6 -> 253.1 mm
Other:
- board text added: "Rev 3.1"
- board text removed: "Rev 2.1"

Commit message: Fixes to PiHatPro pcb board
Other:
- board text added: "Rev 3.2"
- board text removed: "Rev 3.1"
Changed lines of the file:
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@@
     (thickness 1.6)
     (drawings 5)
-    (tracks 120)
+    (tracks 121)
     (zones 0)
     (modules 11)
@@
     (visible_elements FFFEF97F)
     (pcbplotparams
-      (layerselection 0x010f0_fffffff9)
+      (layerselection 0x01020_fffffff9)
       (usegerberextensions false)
       (usegerberattributes true)
@@
     )
   )
-  (gr_text "Rev 3.1" (at 15.36 71.136) (layer F.SilkS)
+  (gr_text "Rev 3.2" (at 15.36 71.136) (layer F.SilkS)
     (effects (font (size 1 1) (thickness 0.15)))
   )
@@
   (segment (start 53.41 23.386) (end 53.41 21.136) (width 1.25) (layer In1.Cu) (net 2))
   (segment (start 53.46 21.036) (end 53.56 20.936) (width 1.5) (layer F.Cu) (net 2))
-  (segment (start 38.76 25.936) (end 40.46 25.936) (width 1.5) (layer F.Cu) (net 2))
   (segment (start 48.16 18.236) (end 52.76 18.236) (width 1.5) (layer B.Cu) (net 2))
   (segment (start 53.46 18.936) (end 53.46 21.036) (width 1.5) (layer B.Cu) (net 2))
@@
   (segment (start 30.26 29.936) (end 34.26 25.936) (width 1.5) (layer B.Cu) (net 2))
   (segment (start 16.46 29.936) (end 30.26 29.936) (width 1.5) (layer B.Cu) (net 2))
+  (segment (start 39.06 25.936) (end 38.96 26.036) (width 1.5) (layer B.Cu) (net 2))
+  (segment (start 40.46 25.936) (end 39.06 25.936) (width 1.5) (layer B.Cu) (net 2))
   (segment (start 28.66 25.936) (end 28.66 25.836) (width 1.5) (layer F.Cu) (net 16))
   (segment (start 25.16 22.336) (end 21.86 22.336) (width 1.5) (layer B.Cu) (net 16))
